Commit message: sliding columns no working

File: urdf_files/sliding_column.urdf (robot description, URDF)
Before this commit: robot column, 1 links, 0 joints
Links:
- link base: mass 10.0 -> 0

Commit message: testing branch

File: urdf_files/sliding_column.urdf (robot description, URDF)
Before this commit: robot sliding_column, 1 links, 0 joints
Links:
- link base: geometry collision cylinder length=1.5 radius=0.3; visual cylinder length=1.5 radius=0.3
